Commit message: transfer to aliyun

File: assets/embodiments/ARX-X5/X5A.urdf (robot description, URDF)
Before this commit: robot X5A, 11 links, 10 joints
Joints:
- joint hand_to_camera_mount: origin xyz=0.057 0 0 rpy=0 0 -3.1416 -> xyz=0.01 0 0.01 rpy=0 0 -3.1416

File: assets/embodiments/franka-panda/panda.urdf (robot description, URDF)
Before this commit: robot panda, 14 links, 13 joints
Joints:
- joint camera_joint: origin xyz=0.042 -0.045 0.0 rpy=1.57079632679 0 -0 -> xyz=0.042 -0.055 0.0 rpy=1.57079632679 0 0.3

File: assets/embodiments/piper/piper.urdf (robot description, URDF)
Before this commit: robot piper_description, 11 links, 10 joints
Joints:
- joint camera_joint: origin xyz=0.032 0.055 0.115 rpy=0 -1.1116926535897932 -1.5707963267948966 -> xyz=0.012 0.06 0.115 rpy=0 -1.1116926535897932 -1.5707963267948966

File: assets/embodiments/ur5-wsg/ur5_wsg_gripper.urdf (robot description, URDF)
Before this commit: robot ur5, 18 links, 17 joints
Joints:
- joint hand_to_camera_mount: origin xyz=0.0 0.08 0 rpy=3.14159265359 1.57079632679 1.57079632679 -> xyz=0.0 0.1 0.04 rpy=3.14159265359 2.2 1.57079632679
